Commit message: add all tasks, mt1, ml1, mt4, ml4, mt/ml algo

File: assets/mjcf/door/mobility.urdf (robot description, URDF)
Before this commit: robot partnet_5b844d6f4d064a52ce6c3e73b818a2cc, 4 links, 3 joints
Links:
- link link_1: geometry collision mesh filename=textured_objs/original-10.obj scale=2 2 2; collision mesh filename=textured_objs/original-11.obj scale=2 2 2
- link link_2: geometry collision mesh filename=textured_objs/original-5.obj scale=2 2 2; collision mesh filename=textured_objs/original-6.obj scale=2 2 2
Joints:
- joint joint_1: origin xyz=-0.4165270657166128 0.48329200000000005 0.008461858680020029 -> xyz=-0.4265270657166128 0.48329200000000005 0.008461858680020029
